Commit message: Этап 5: сцена с рельсами, граница по глубине и автомат заезда
Стенд собран по обмеру, а не по догадке: труба Ø51 мм, колея 545 мм,
настил 120 мм, конец рельсов — буква П с радиусом 145 мм и вылетом
210 мм на настил. Размеры сняты с ортофото из датасета RealSense, а не
взяты из каталога. Ключевая величина здесь одна: разность радиуса
колеса 101.4 мм и радиуса ролика 50.0 мм даёт 51.4 мм против трубы
51 мм, то есть ступенька при переходе 0.4 мм и от высоты настила не
зависит.

Граница настила находится по глубине геометрически, а не эвристикой по
сетке. Для каждого пикселя считается, на какой дальности луч встретил бы
опорную плоскость; если измеренная глубина заметно больше, луч перелетел
край. Допуск привязан к шуму дальномера, который растёт как квадрат
дальности. Точность 3 мм при дрожании 0.2 мм.

Облако отдаётся в кадре КАМЕРЫ, а не робота. RTAB-Map берёт начало
кадра облака за точку наблюдения и трассирует лучи оттуда: в кадре
робота он считал сенсор стоящим под роботом на уровне пола и расчищал
свободным всё вокруг, включая площадь ПОД роботом, которую камера
физически не видит.

Нижний уровень в облако не идёт вовсе. Подтягивать его к опорной
плоскости неверно: площадь за краем настила ложилась СВОБОДНОЙ, и
удерживала планировщик одна тонкая линия края, а она рвётся — замерено,
на метре от робота кромка закрыта на 100 %, на двух на 42 %. Без точек
клетки остаются неизвестными, а неизвестность для Nav2 непроезжая.

Сегментация рельсов пока подменена оракулом по истинной геометрии мира.
Интерфейс выбран такой же, какой вернёт модель CV: маска в кадре камеры.
Маска строится через буфер дальности, а не диском по осевой линии —
камера смотрит сверху под углом и видит верх и ближний бок трубы, с
чистым диском 10 % пикселей оставались снаружи, а раздутый диск
перехлёстывал на пол за кромкой и ронял долю попаданий с 95 до 71 %.
Итог: маска накрывает 98.7 % пикселей трубы, размах −297..+301 мм при
осях ±272.

Цвет карты везётся в самих точках: RTAB-Map сливает кромку, рельсы и
прочее в одно облако, и слой в RViz красится целиком. Кромка красная,
рельсы зелёные. Точки пола ближе 10 см к рельсу выброшены — сетка
усредняет цвет в вокселе 5 см, и труба 51 мм внутри клетки 50 мм всегда
в меньшинстве, вместо зелёного выходило (125,207,142).

Автомат заезда: ОСМОТР, ПОИСК, ПОДХОД, ВЫВЕРКА, ЗАЕЗД, ОТКАТ с
повтором. Nav2 ведёт только подход по настилу. Сам заезд идёт напрямую,
потому что на рельсах радиус качения падает вдвое и регулятор, считающий
это отставанием, начал бы разгоняться. Успех определяется одним
признаком: продвигается робот или стоит. Правильную скорость знать не
нужно и вредно — при заезде робот подкренивается и может застрять.

Замерено на случайных позах: заезд удаётся с первой попытки, финиш на
2.4 м по трубам, поперечное смещение в пределах 8.6 мм при допуске 18,
курс 0.2°. В журнале прямо виден переход на рельсы: до него 108-119 мм
за секундное окно при команде 120, после — 68-77.

Nav2 настроен полигоном 1.22 x 0.90 м, а не окружностью: описанный
радиус 0.775 м не оставил бы на настиле 2 x 3 м ни одной свободной
клетки под центр робота. Поднимается после контроллеров — его менеджер
жизненного цикла не дожидался ответа серверов, пока рядом стартовали
Gazebo и RTAB-Map, и бросал подъём на полпути.

Площадь под роботом детектор доклеивает сам: камера видит с 0.6 м, эта
клетка не наблюдается никогда, а неизвестность непроезжая — планировщик
отказывался строить путь от такого старта. Пятачок намеренно меньше
корпуса и равен колёсному прямоугольнику: корпус свисает за колёса на
0.28 м, и у кромки этот свес висит над обрывом.

Co-Authored-By: Claude Opus 5 <noreply@anthropic.com>

File: src/maze_nav/urdf/agro_robot.urdf.xacro (robot description, xacro)
@@ -45,19 +45,34 @@
       scale="0.001 0.001 0.001"/></geometry>
       <material name="hub"/></visual>
-    <!-- Коллизия рельсового ролика: ДВА цилиндра вместо меша.
-         Профиль с канавкой невыпуклый, а движки быстро считают
-         только выпуклые тела. Пара "дорожка + реборда" — это две
-         выпуклые формы, вместе дающие ступеньку: рельса
-         удерживается сбоку, но соскочить при перекосе можно,
-         а это и есть предмет изучения на заезде.
-         Чего пара не даёт — плавности галтели: переход выйдет
-         ступенькой. Если заезд поведёт себя странно, смотреть сюда. -->
-    <collision><!-- дорожка -->
-      <origin xyz="0 -0.0837 0" rpy="1.570796 0 0"/>
-      <geometry><cylinder radius="0.05" length="0.0423"/></geometry>
-    </collision>
-    <collision><!-- реборда -->
-      <origin xyz="0 -0.0513 0" rpy="1.570796 0 0"/>
-      <geometry><cylinder radius="0.075" length="0.0227"/></geometry>
+    <!-- Коллизия рельсового ролика: набор цилиндров по измеренному
+         профилю (см. RAIL_PROFILE). Канавка вогнутая, одним телом
+         её не посчитать — движки берут только выпуклые формы. -->
+    <collision><!-- R=50.0 мм -->
+      <origin xyz="0 -0.0849 0" rpy="1.570796 0 0"/>
+      <geometry><cylinder radius="0.05" length="0.0399"/></geometry>
+    </collision>
+    <collision><!-- R=52.0 мм -->
+      <origin xyz="0 -0.0625 0" rpy="1.570796 0 0"/>
+      <geometry><cylinder radius="0.052" length="0.0050"/></geometry>
+    </collision>
+    <collision><!-- R=55.0 мм -->
+      <origin xyz="0 -0.0580 0" rpy="1.570796 0 0"/>
+      <geometry><cylinder radius="0.055" length="0.0040"/></geometry>
+    </collision>
+    <collision><!-- R=58.0 мм -->
+      <origin xyz="0 -0.0545 0" rpy="1.570796 0 0"/>
+      <geometry><cylinder radius="0.058" length="0.0030"/></geometry>
+    </collision>
+    <collision><!-- R=62.0 мм -->
+      <origin xyz="0 -0.0515 0" rpy="1.570796 0 0"/>
+      <geometry><cylinder radius="0.062" length="0.0030"/></geometry>
+    </collision>
+    <collision><!-- R=68.0 мм -->
+      <origin xyz="0 -0.0485 0" rpy="1.570796 0 0"/>
+      <geometry><cylinder radius="0.068" length="0.0030"/></geometry>
+    </collision>
+    <collision><!-- R=75.0 мм -->
+      <origin xyz="0 -0.0435 0" rpy="1.570796 0 0"/>
+      <geometry><cylinder radius="0.075" length="0.0071"/></geometry>
     </collision>
   </link>
@@ -250,19 +265,34 @@
       scale="0.001 0.001 0.001"/></geometry>
       <material name="hub"/></visual>
-    <!-- Коллизия рельсового ролика: ДВА цилиндра вместо меша.
-         Профиль с канавкой невыпуклый, а движки быстро считают
-         только выпуклые тела. Пара "дорожка + реборда" — это две
-         выпуклые формы, вместе дающие ступеньку: рельса
-         удерживается сбоку, но соскочить при перекосе можно,
-         а это и есть предмет изучения на заезде.
-         Чего пара не даёт — плавности галтели: переход выйдет
-         ступенькой. Если заезд поведёт себя странно, смотреть сюда. -->
-    <collision><!-- дорожка -->
-      <origin xyz="0 0.0837 0" rpy="1.570796 0 0"/>
-      <geometry><cylinder radius="0.05" length="0.0423"/></geometry>
-    </collision>
-    <collision><!-- реборда -->
-      <origin xyz="0 0.0513 0" rpy="1.570796 0 0"/>
-      <geometry><cylinder radius="0.075" length="0.0227"/></geometry>
+    <!-- Коллизия рельсового ролика: набор цилиндров по измеренному
+         профилю (см. RAIL_PROFILE). Канавка вогнутая, одним телом
+         её не посчитать — движки берут только выпуклые формы. -->
+    <collision><!-- R=50.0 мм -->
+      <origin xyz="0 0.0849 0" rpy="1.570796 0 0"/>
+      <geometry><cylinder radius="0.05" length="0.0399"/></geometry>
+    </collision>
+    <collision><!-- R=52.0 мм -->
+      <origin xyz="0 0.0625 0" rpy="1.570796 0 0"/>
+      <geometry><cylinder radius="0.052" length="0.0050"/></geometry>
+    </collision>
+    <collision><!-- R=55.0 мм -->
+      <origin xyz="0 0.0580 0" rpy="1.570796 0 0"/>
+      <geometry><cylinder radius="0.055" length="0.0040"/></geometry>
+    </collision>
+    <collision><!-- R=58.0 мм -->
+      <origin xyz="0 0.0545 0" rpy="1.570796 0 0"/>
+      <geometry><cylinder radius="0.058" length="0.0030"/></geometry>
+    </collision>
+    <collision><!-- R=62.0 мм -->
+      <origin xyz="0 0.0515 0" rpy="1.570796 0 0"/>
+      <geometry><cylinder radius="0.062" length="0.0030"/></geometry>
+    </collision>
+    <collision><!-- R=68.0 мм -->
+      <origin xyz="0 0.0485 0" rpy="1.570796 0 0"/>
+      <geometry><cylinder radius="0.068" length="0.0030"/></geometry>
+    </collision>
+    <collision><!-- R=75.0 мм -->
+      <origin xyz="0 0.0435 0" rpy="1.570796 0 0"/>
+      <geometry><cylinder radius="0.075" length="0.0071"/></geometry>
     </collision>
   </link>
@@ -455,19 +485,34 @@
       scale="0.001 0.001 0.001"/></geometry>
       <material name="hub"/></visual>
-    <!-- Коллизия рельсового ролика: ДВА цилиндра вместо меша.
-         Профиль с канавкой невыпуклый, а движки быстро считают
-         только выпуклые тела. Пара "дорожка + реборда" — это две
-         выпуклые формы, вместе дающие ступеньку: рельса
-         удерживается сбоку, но соскочить при перекосе можно,
-         а это и есть предмет изучения на заезде.
-         Чего пара не даёт — плавности галтели: переход выйдет
-         ступенькой. Если заезд поведёт себя странно, смотреть сюда. -->
-    <collision><!-- дорожка -->
-      <origin xyz="0 -0.0837 0" rpy="1.570796 0 0"/>
-      <geometry><cylinder radius="0.05" length="0.0423"/></geometry>
-    </collision>
-    <collision><!-- реборда -->
-      <origin xyz="0 -0.0513 0" rpy="1.570796 0 0"/>
-      <geometry><cylinder radius="0.075" length="0.0227"/></geometry>
+    <!-- Коллизия рельсового ролика: набор цилиндров по измеренному
+         профилю (см. RAIL_PROFILE). Канавка вогнутая, одним телом
+         её не посчитать — движки берут только выпуклые формы. -->
+    <collision><!-- R=50.0 мм -->
+      <origin xyz="0 -0.0849 0" rpy="1.570796 0 0"/>
+      <geometry><cylinder radius="0.05" length="0.0399"/></geometry>
+    </collision>
+    <collision><!-- R=52.0 мм -->
+      <origin xyz="0 -0.0625 0" rpy="1.570796 0 0"/>
+      <geometry><cylinder radius="0.052" length="0.0050"/></geometry>
+    </collision>
+    <collision><!-- R=55.0 мм -->
+      <origin xyz="0 -0.0580 0" rpy="1.570796 0 0"/>
+      <geometry><cylinder radius="0.055" length="0.0040"/></geometry>
+    </collision>
+    <collision><!-- R=58.0 мм -->
+      <origin xyz="0 -0.0545 0" rpy="1.570796 0 0"/>
+      <geometry><cylinder radius="0.058" length="0.0030"/></geometry>
+    </collision>
+    <collision><!-- R=62.0 мм -->
+      <origin xyz="0 -0.0515 0" rpy="1.570796 0 0"/>
+      <geometry><cylinder radius="0.062" length="0.0030"/></geometry>
+    </collision>
+    <collision><!-- R=68.0 мм -->
+      <origin xyz="0 -0.0485 0" rpy="1.570796 0 0"/>
+      <geometry><cylinder radius="0.068" length="0.0030"/></geometry>
+    </collision>
+    <collision><!-- R=75.0 мм -->
+      <origin xyz="0 -0.0435 0" rpy="1.570796 0 0"/>
+      <geometry><cylinder radius="0.075" length="0.0071"/></geometry>
     </collision>
   </link>
@@ -660,19 +705,34 @@
       scale="0.001 0.001 0.001"/></geometry>
       <material name="hub"/></visual>
-    <!-- Коллизия рельсового ролика: ДВА цилиндра вместо меша.
-         Профиль с канавкой невыпуклый, а движки быстро считают
-         только выпуклые тела. Пара "дорожка + реборда" — это две
-         выпуклые формы, вместе дающие ступеньку: рельса
-         удерживается сбоку, но соскочить при перекосе можно,
-         а это и есть предмет изучения на заезде.
-         Чего пара не даёт — плавности галтели: переход выйдет
-         ступенькой. Если заезд поведёт себя странно, смотреть сюда. -->
-    <collision><!-- дорожка -->
-      <origin xyz="0 0.0837 0" rpy="1.570796 0 0"/>
-      <geometry><cylinder radius="0.05" length="0.0423"/></geometry>
-    </collision>
-    <collision><!-- реборда -->
-      <origin xyz="0 0.0513 0" rpy="1.570796 0 0"/>
-      <geometry><cylinder radius="0.075" length="0.0227"/></geometry>
+    <!-- Коллизия рельсового ролика: набор цилиндров по измеренному
+         профилю (см. RAIL_PROFILE). Канавка вогнутая, одним телом
+         её не посчитать — движки берут только выпуклые формы. -->
+    <collision><!-- R=50.0 мм -->
+      <origin xyz="0 0.0849 0" rpy="1.570796 0 0"/>
+      <geometry><cylinder radius="0.05" length="0.0399"/></geometry>
+    </collision>
+    <collision><!-- R=52.0 мм -->
+      <origin xyz="0 0.0625 0" rpy="1.570796 0 0"/>
+      <geometry><cylinder radius="0.052" length="0.0050"/></geometry>
+    </collision>
+    <collision><!-- R=55.0 мм -->
+      <origin xyz="0 0.0580 0" rpy="1.570796 0 0"/>
+      <geometry><cylinder radius="0.055" length="0.0040"/></geometry>
+    </collision>
+    <collision><!-- R=58.0 мм -->
+      <origin xyz="0 0.0545 0" rpy="1.570796 0 0"/>
+      <geometry><cylinder radius="0.058" length="0.0030"/></geometry>
+    </collision>
+    <collision><!-- R=62.0 мм -->
+      <origin xyz="0 0.0515 0" rpy="1.570796 0 0"/>
+      <geometry><cylinder radius="0.062" length="0.0030"/></geometry>
+    </collision>
+    <collision><!-- R=68.0 мм -->
+      <origin xyz="0 0.0485 0" rpy="1.570796 0 0"/>
+      <geometry><cylinder radius="0.068" length="0.0030"/></geometry>
+    </collision>
+    <collision><!-- R=75.0 мм -->
+      <origin xyz="0 0.0435 0" rpy="1.570796 0 0"/>
+      <geometry><cylinder radius="0.075" length="0.0071"/></geometry>
     </collision>
   </link>
@@ -1069,9 +1129,29 @@
     <mu1>0.2</mu1><mu2>0.2</mu2>
   </gazebo>
-  <link name="camera_link"/>
+  <!-- Кронштейн: от профиля крыши ВПЕРЁД, горизонтально.
+       Наклон живёт отдельно, в camera_link, чтобы менять его одной
+       константой, не трогая вынос. -->
+  <link name="camera_mount_link">
+    <visual><origin xyz="-0.0500 0 0" rpy="0 1.570796 0"/>
+      <geometry><cylinder radius="0.012" length="0.1"/></geometry>
+      <material name="hub"/></visual>
+  </link>
+  <joint name="camera_mount_joint" type="fixed">
+    <parent link="base_link"/><child link="camera_mount_link"/>
+    <origin xyz="0.5000 0.0 0.6147"/>
+  </joint>
+  <!-- D435, наклон 30° вниз -->
+  <link name="camera_link">
+    <visual><geometry><box size="0.025 0.090 0.025"/></geometry>
+      <material name="hub"/></visual>
+  </link>
   <joint name="camera_joint" type="fixed">
-    <parent link="base_link"/><child link="camera_link"/>
-    <origin xyz="0.60 0 0.63"/>
-  </joint>
+    <parent link="camera_mount_link"/><child link="camera_link"/>
+    <origin rpy="0 0.523599 0"/>
+  </joint>
+  <!-- Оптический кадр: z вперёд, x вправо, y вниз — как принято в ROS.
+       Именно его имя должно стоять в gz_frame_id ниже, иначе Gazebo
+       проштампует снимки составным именем вида model/link/sensor,
+       которого нет в TF, и SLAM молча развалится. -->
   <link name="camera_depth_optical_frame"/>
   <joint name="camera_optical_joint" type="fixed">
@@ -1079,7 +1159,42 @@
     <origin rpy="-1.570796 0 -1.570796"/>
   </joint>
+  <gazebo reference="camera_link">
+    <sensor name="d435" type="rgbd_camera">
+      <update_rate>15</update_rate>
+      <always_on>1</always_on>
+      <topic>camera</topic>
+      <gz_frame_id>camera_depth_optical_frame</gz_frame_id>
+      <camera>
+        <horizontal_fov>1.518436</horizontal_fov>
+        <image><width>640</width><height>480</height>
+          <format>R8G8B8</format></image>
+        <clip><near>0.28</near><far>10.0</far></clip>
+        <optical_frame_id>camera_depth_optical_frame</optical_frame_id>
+      </camera>
+    </sensor>
+  </gazebo>
+  <!-- Стоит в начале base_link: центр колёсной базы на высоте оси.
+       Место выбрано не для удобства. Гироскоп от положения не
+       зависит вовсе — угловая скорость у твёрдого тела одинакова
+       везде. А вот акселерометр, смещённый на r от центра вращения,
+       ловит при повороте центростремительное w^2*r и тангенциальное
+       a*r. При r=0.5 м и w=0.5 рад/с это 0.125 м/с2 — вектор
+       гравитации наклоняется на 0.7°, а из него берутся крен и
+       тангаж. robot_localization поворачивает данные по TF, но
+       вынос плеча НЕ компенсирует, так что одним объявлением
+       положения тут не отделаться.
+       Нам крен нужен чистым: по нему отличается правильная посадка
+       на дорожку качения от заезда на галтель. -->
   <link name="imu_link"/>
   <joint name="imu_joint" type="fixed">
     <parent link="base_link"/><child link="imu_link"/><origin xyz="0 0 0"/>
   </joint>
+  <gazebo reference="imu_link">
+    <sensor name="imu" type="imu">
+      <update_rate>100</update_rate>
+      <always_on>1</always_on>
+      <topic>imu</topic>
+      <gz_frame_id>imu_link</gz_frame_id>
+    </sensor>
+  </gazebo>
 </robot>
