Commit message: Этап 6: перенос на реального робота — ИНС, камера и опорная плоскость
Вычисления идут на ноутбуке, который стоит на самом роботе: к нему
подключены RealSense D435i и ИНС, а наружу уходит только /cmd_nav по
сети через ROS_DOMAIN_ID. Разные дистрибутивы помехой не оказались —
Jazzy на ноутбуке и Humble на роботе обмениваются штатными сообщениями
без переходника, проверено на geometry_msgs/Twist.

ИНС собрана на Pico с MPU6050, прошивка переделана из дипломного стенда
и лежит в корне проекта. FIFO убран, хотя на стенде он использовался: у
него нет меток границ пакета, и однажды сбившееся чтение едет со
смещением НАВСЕГДА. Замерено на живой плате — лежащий плашмя датчик
отдавал тяжесть по x, тогда как прямое чтение регистров показывало её
по z, расхождение 10.3 м/с². Выравнивание сбросом при запуске проблему
не снимало: проверка проходила, а на ходу выравнивание терялось.

Узел ИНС срезает накопленное отставание. Порт читается по таймеру, и
пока узел один, буфер пуст. Но под полной нагрузкой — камера, RTAB-Map,
Nav2, детектор края — таймеру перестаёт хватать процессора, и выборки
копятся в буфере ядра. Метки у них при этом ЧЕСТНЫЕ, прошивка ставит
время съёма, поэтому отставание целиком переходит в метки: замерено
около 40 мс, и rgbd_odometry бросал каждый кадр подряд. Старые выборки
одометрии не нужны, ей нужна свежая ориентация.

Опорная плоскость детектора кромки теперь измеряется по ближней земле
под роботом, а не берётся из URDF. В симуляторе URDF и есть истина, и
абсолютный порог работал. На живом роботе камеру крепят руками: в URDF
записан наклон 45°, фактический оказался около 48-50°, и этих градусов
хватило, чтобы настил высотой 10 см лёг на -1 см вместо -10 и не прошёл
порог обрыва -6 см. Детектор при этом молчал совершенно исправно: точки
были, перелёта не было. После подгонки на том же стенде ниже порога
оказалось 72688 точек вместо нуля. Побочно это снимает крен от
подвески, который при камере на крыше даёт на двух метрах те же
сантиметры.

Nav2 обходит монитор столкновений вместо того, чтобы кормить его
облаком камеры: добавление источника нагружало процессор так, что
задержка доходила до 0.9 с, а цикл падал до 10.4 Гц. Пределы скоростей
подняты под ковролин, на котором робот не трогался с места.

Документация приведена в соответствие с сделанным: таблица этапов
отставала на три позиции, а развилка 4.2 разрешена не выбором одного из
трёх вариантов, как предполагалось, а соединением двух — YOLO отвечает
«что из этого рельс», геометрия «где он в метрах».

Co-Authored-By: Claude Opus 5 <noreply@anthropic.com>

File: src/maze_nav/urdf/agro_robot_real.urdf.xacro (robot description, xacro)
@@ -915,231 +915,17 @@
        с полом, и именно поэтому боковое движение возникает
        из физики, а не рисуется кинематикой. -->
-  <ros2_control name="GazeboSystem" type="system">
-    <hardware>
-      <plugin>gz_ros2_control/GazeboSimSystem</plugin>
-    </hardware>
-    <joint name="fl_wheel_joint">
-      <!-- Мотор-колесо с редуктором управляется скоростью,
-           поэтому командный интерфейс velocity, а не effort:
-           иначе поведение на проскальзывании будет непохожим. -->
-      <command_interface name="velocity">
-        <param name="min">-20.0</param>
-        <param name="max">20.0</param>
-      </command_interface>
-      <state_interface name="position"/>
-      <state_interface name="velocity"/>
-    </joint>
-    <joint name="fr_wheel_joint">
-      <!-- Мотор-колесо с редуктором управляется скоростью,
-           поэтому командный интерфейс velocity, а не effort:
-           иначе поведение на проскальзывании будет непохожим. -->
-      <command_interface name="velocity">
-        <param name="min">-20.0</param>
-        <param name="max">20.0</param>
-      </command_interface>
-      <state_interface name="position"/>
-      <state_interface name="velocity"/>
-    </joint>
-    <joint name="rl_wheel_joint">
-      <!-- Мотор-колесо с редуктором управляется скоростью,
-           поэтому командный интерфейс velocity, а не effort:
-           иначе поведение на проскальзывании будет непохожим. -->
-      <command_interface name="velocity">
-        <param name="min">-20.0</param>
-        <param name="max">20.0</param>
-      </command_interface>
-      <state_interface name="position"/>
-      <state_interface name="velocity"/>
-    </joint>
-    <joint name="rr_wheel_joint">
-      <!-- Мотор-колесо с редуктором управляется скоростью,
-           поэтому командный интерфейс velocity, а не effort:
-           иначе поведение на проскальзывании будет непохожим. -->
-      <command_interface name="velocity">
-        <param name="min">-20.0</param>
-        <param name="max">20.0</param>
-      </command_interface>
-      <state_interface name="position"/>
-      <state_interface name="velocity"/>
-    </joint>
-  </ros2_control>
-  <gazebo>
-    <plugin filename="gz_ros2_control-system"
-            name="gz_ros2_control::GazeboSimROS2ControlPlugin">
-      <parameters>$(find maze_nav)/params/agro_controllers.yaml</parameters>
-    </plugin>
-  </gazebo>
-  <gazebo reference="fl_roller_0">
-    <mu1>1.0</mu1><mu2>1.0</mu2>
-  </gazebo>
-  <gazebo reference="fl_roller_1">
-    <mu1>1.0</mu1><mu2>1.0</mu2>
-  </gazebo>
-  <gazebo reference="fl_roller_2">
-    <mu1>1.0</mu1><mu2>1.0</mu2>
-  </gazebo>
-  <gazebo reference="fl_roller_3">
-    <mu1>1.0</mu1><mu2>1.0</mu2>
-  </gazebo>
-  <gazebo reference="fl_roller_4">
-    <mu1>1.0</mu1><mu2>1.0</mu2>
-  </gazebo>
-  <gazebo reference="fl_roller_5">
-    <mu1>1.0</mu1><mu2>1.0</mu2>
-  </gazebo>
-  <gazebo reference="fl_roller_6">
-    <mu1>1.0</mu1><mu2>1.0</mu2>
-  </gazebo>
-  <gazebo reference="fl_roller_7">
-    <mu1>1.0</mu1><mu2>1.0</mu2>
-  </gazebo>
-  <gazebo reference="fl_roller_8">
-    <mu1>1.0</mu1><mu2>1.0</mu2>
-  </gazebo>
-  <gazebo reference="fl_roller_9">
-    <mu1>1.0</mu1><mu2>1.0</mu2>
-  </gazebo>
-  <gazebo reference="fl_roller_10">
-    <mu1>1.0</mu1><mu2>1.0</mu2>
-  </gazebo>
-  <gazebo reference="fl_roller_11">
-    <mu1>1.0</mu1><mu2>1.0</mu2>
-  </gazebo>
-  <gazebo reference="fl_wheel">
-    <mu1>1.0</mu1><mu2>1.0</mu2>
-  </gazebo>
-  <gazebo reference="fr_roller_0">
-    <mu1>1.0</mu1><mu2>1.0</mu2>
-  </gazebo>
-  <gazebo reference="fr_roller_1">
-    <mu1>1.0</mu1><mu2>1.0</mu2>
-  </gazebo>
-  <gazebo reference="fr_roller_2">
-    <mu1>1.0</mu1><mu2>1.0</mu2>
-  </gazebo>
-  <gazebo reference="fr_roller_3">
-    <mu1>1.0</mu1><mu2>1.0</mu2>
-  </gazebo>
-  <gazebo reference="fr_roller_4">
-    <mu1>1.0</mu1><mu2>1.0</mu2>
-  </gazebo>
-  <gazebo reference="fr_roller_5">
-    <mu1>1.0</mu1><mu2>1.0</mu2>
-  </gazebo>
-  <gazebo reference="fr_roller_6">
-    <mu1>1.0</mu1><mu2>1.0</mu2>
-  </gazebo>
-  <gazebo reference="fr_roller_7">
-    <mu1>1.0</mu1><mu2>1.0</mu2>
-  </gazebo>
-  <gazebo reference="fr_roller_8">
-    <mu1>1.0</mu1><mu2>1.0</mu2>
-  </gazebo>
-  <gazebo reference="fr_roller_9">
-    <mu1>1.0</mu1><mu2>1.0</mu2>
-  </gazebo>
-  <gazebo reference="fr_roller_10">
-    <mu1>1.0</mu1><mu2>1.0</mu2>
-  </gazebo>
-  <gazebo reference="fr_roller_11">
-    <mu1>1.0</mu1><mu2>1.0</mu2>
-  </gazebo>
-  <gazebo reference="fr_wheel">
-    <mu1>1.0</mu1><mu2>1.0</mu2>
-  </gazebo>
-  <gazebo reference="rl_roller_0">
-    <mu1>1.0</mu1><mu2>1.0</mu2>
-  </gazebo>
-  <gazebo reference="rl_roller_1">
-    <mu1>1.0</mu1><mu2>1.0</mu2>
-  </gazebo>
-  <gazebo reference="rl_roller_2">
-    <mu1>1.0</mu1><mu2>1.0</mu2>
-  </gazebo>
-  <gazebo reference="rl_roller_3">
-    <mu1>1.0</mu1><mu2>1.0</mu2>
-  </gazebo>
-  <gazebo reference="rl_roller_4">
-    <mu1>1.0</mu1><mu2>1.0</mu2>
-  </gazebo>
-  <gazebo reference="rl_roller_5">
-    <mu1>1.0</mu1><mu2>1.0</mu2>
-  </gazebo>
-  <gazebo reference="rl_roller_6">
-    <mu1>1.0</mu1><mu2>1.0</mu2>
-  </gazebo>
-  <gazebo reference="rl_roller_7">
-    <mu1>1.0</mu1><mu2>1.0</mu2>
-  </gazebo>
-  <gazebo reference="rl_roller_8">
-    <mu1>1.0</mu1><mu2>1.0</mu2>
-  </gazebo>
-  <gazebo reference="rl_roller_9">
-    <mu1>1.0</mu1><mu2>1.0</mu2>
-  </gazebo>
-  <gazebo reference="rl_roller_10">
-    <mu1>1.0</mu1><mu2>1.0</mu2>
-  </gazebo>
-  <gazebo reference="rl_roller_11">
-    <mu1>1.0</mu1><mu2>1.0</mu2>
-  </gazebo>
-  <gazebo reference="rl_wheel">
-    <mu1>1.0</mu1><mu2>1.0</mu2>
-  </gazebo>
-  <gazebo reference="rr_roller_0">
-    <mu1>1.0</mu1><mu2>1.0</mu2>
-  </gazebo>
-  <gazebo reference="rr_roller_1">
-    <mu1>1.0</mu1><mu2>1.0</mu2>
-  </gazebo>
-  <gazebo reference="rr_roller_2">
-    <mu1>1.0</mu1><mu2>1.0</mu2>
-  </gazebo>
-  <gazebo reference="rr_roller_3">
-    <mu1>1.0</mu1><mu2>1.0</mu2>
-  </gazebo>
-  <gazebo reference="rr_roller_4">
-    <mu1>1.0</mu1><mu2>1.0</mu2>
-  </gazebo>
-  <gazebo reference="rr_roller_5">
-    <mu1>1.0</mu1><mu2>1.0</mu2>
-  </gazebo>
-  <gazebo reference="rr_roller_6">
-    <mu1>1.0</mu1><mu2>1.0</mu2>
-  </gazebo>
-  <gazebo reference="rr_roller_7">
-    <mu1>1.0</mu1><mu2>1.0</mu2>
-  </gazebo>
-  <gazebo reference="rr_roller_8">
-    <mu1>1.0</mu1><mu2>1.0</mu2>
-  </gazebo>
-  <gazebo reference="rr_roller_9">
-    <mu1>1.0</mu1><mu2>1.0</mu2>
-  </gazebo>
-  <gazebo reference="rr_roller_10">
-    <mu1>1.0</mu1><mu2>1.0</mu2>
-  </gazebo>
-  <gazebo reference="rr_roller_11">
-    <mu1>1.0</mu1><mu2>1.0</mu2>
-  </gazebo>
-  <gazebo reference="rr_wheel">
-    <mu1>1.0</mu1><mu2>1.0</mu2>
-  </gazebo>
-  <gazebo reference="base_link">
-    <mu1>0.2</mu1><mu2>0.2</mu2>
-  </gazebo>
   <!-- Кронштейн: от профиля крыши ВПЕРЁД, горизонтально.
        Наклон живёт отдельно, в camera_link, чтобы менять его одной
        константой, не трогая вынос. -->
   <link name="camera_mount_link">
-    <visual><origin xyz="-0.0500 0 0" rpy="0 1.570796 0"/>
-      <geometry><cylinder radius="0.012" length="0.1"/></geometry>
+    <visual><origin xyz="-0.0400 0 0" rpy="0 1.570796 0"/>
+      <geometry><cylinder radius="0.012" length="0.08"/></geometry>
       <material name="hub"/></visual>
   </link>
   <joint name="camera_mount_joint" type="fixed">
     <parent link="base_link"/><child link="camera_mount_link"/>
-    <origin xyz="0.5000 0.0 0.6147"/>
-  </joint>
-  <!-- D435, наклон 30° вниз -->
+    <origin xyz="0.4905 0.0 0.6747000000000001"/>
+  </joint>
+  <!-- D435, наклон 45° вниз -->
   <link name="camera_link">
     <visual><geometry><box size="0.025 0.090 0.025"/></geometry>
@@ -1148,30 +934,6 @@
   <joint name="camera_joint" type="fixed">
     <parent link="camera_mount_link"/><child link="camera_link"/>
-    <origin rpy="0 0.523599 0"/>
-  </joint>
-  <!-- Оптический кадр: z вперёд, x вправо, y вниз — как в ROS.
-       Именно его имя должно стоять в gz_frame_id ниже, иначе
-       Gazebo проштампует снимки составным именем вида
-       model/link/sensor, которого нет в TF, и SLAM развалится. -->
-  <link name="camera_depth_optical_frame"/>
-  <joint name="camera_optical_joint" type="fixed">
-    <parent link="camera_link"/><child link="camera_depth_optical_frame"/>
-    <origin rpy="-1.570796 0 -1.570796"/>
-  </joint>
-  <gazebo reference="camera_link">
-    <sensor name="d435" type="rgbd_camera">
-      <update_rate>15</update_rate>
-      <always_on>1</always_on>
-      <topic>camera</topic>
-      <gz_frame_id>camera_depth_optical_frame</gz_frame_id>
-      <camera>
-        <horizontal_fov>1.518436</horizontal_fov>
-        <image><width>640</width><height>480</height>
-          <format>R8G8B8</format></image>
-        <clip><near>0.28</near><far>10.0</far></clip>
-        <optical_frame_id>camera_depth_optical_frame</optical_frame_id>
-      </camera>
-    </sensor>
-  </gazebo>
+    <origin rpy="0 0.785398 0"/>
+  </joint>
   <!-- Стоит в начале base_link: центр колёсной базы на высоте оси.
        Место выбрано не для удобства. Гироскоп от положения не
@@ -1190,11 +952,3 @@
     <parent link="base_link"/><child link="imu_link"/><origin xyz="0 0 0"/>
   </joint>
-  <gazebo reference="imu_link">
-    <sensor name="imu" type="imu">
-      <update_rate>100</update_rate>
-      <always_on>1</always_on>
-      <topic>imu</topic>
-      <gz_frame_id>imu_link</gz_frame_id>
-    </sensor>
-  </gazebo>
 </robot>

Commit message: Калибровка камеры по её собственной ИНС: угол 50.1, высота 723 мм
Три помощника замера вместо догадок о том, как стоит камера.

cam_pitch.py меряет наклон по акселерометру самой камеры, без карты
глубины и без TF: неподвижный датчик показывает направление «вверх», и
этого довольно. После пересборки робота дал 50.18 градуса при 250
выборках и дрожании 0.018 м/с².

cam_level.py сравнивает нормаль земли по глубине с вертикалью по
тяжести. Угол между ними не зависит от того, ровно ли стоит робот:
наклонится робот — повернутся оба вектора разом.

imu_level.py считает перекос крепления ИНС и выдаёт готовые rpy.

ВЫСОТА КАМЕРЫ ИСПРАВЛЕНА, 776 -> 723 мм. Детектор обрыва печатал, что
подогнанная плоскость настила расходится с URDF на стабильные +53 мм при
наклоне всего 0.50 градуса: угол верен, а камера ниже обещанного.
Рулетка подтвердила — около 720 мм. Из-за этого расхождения накопленный
слой рельсов лежал НИЖЕ текстурной карты примерно на диаметр трубы: слой
строится из облака с поправкой плоскости, а карту RTAB-Map собирает сам
из rgb+depth по URDF и поправки не видит.

В прошивке Pico разбор KeyboardInterrupt по частоте: три прерывания за
секунду считаются намеренным входом в REPL, одиночное — помехой. Плата
трижды замолкала оттого, что прерывание проходило через except Exception.

Co-Authored-By: Claude Opus 5 <noreply@anthropic.com>

File: src/maze_nav/urdf/agro_robot_real.urdf.xacro (robot description, xacro)
@@ -925,7 +925,7 @@
   <joint name="camera_mount_joint" type="fixed">
     <parent link="base_link"/><child link="camera_mount_link"/>
-    <origin xyz="0.4905 0.0 0.6747000000000001"/>
-  </joint>
-  <!-- D435, наклон 45° вниз -->
+    <origin xyz="0.4905 0.0 0.6217"/>
+  </joint>
+  <!-- D435, наклон 50° вниз -->
   <link name="camera_link">
     <visual><geometry><box size="0.025 0.090 0.025"/></geometry>
@@ -934,5 +934,5 @@
   <joint name="camera_joint" type="fixed">
     <parent link="camera_mount_link"/><child link="camera_link"/>
-    <origin rpy="0 0.785398 0"/>
+    <origin rpy="0 0.874410 0"/>
   </joint>
   <!-- Стоит в начале base_link: центр колёсной базы на высоте оси.

Commit message: Камера на стационарном креплении: угол 49, высота минус 58 мм
Угол замерен двумя независимыми способами, и это не перестраховка, а
единственный способ отделить наклон крепления от уклона пола.
Акселерометр камеры (от ТЯЖЕСТИ): 49.05 и 49.08 в двух прогонах по 120
выборок. Плоскость пола из глубины (от ПОЛА), RANSAC и SVD по 369 тысячам
точек с остатком 3.2 мм: 48.98 и 48.97. Совпали они только потому, что
пол горизонтальный и робот стоит ровно. Крен около 0.1 — крепление
квадратное, слагаемого по крену в описании нет.

Высота сперва выглядела противоречием: подгонка плоскости давала 775 мм,
а детектор обрыва печатал «сдвиг +58 мм». Разрешается стендом. Детектор
меряет до настила, на котором стоят КОЛЁСА, а подгонка в тот раз поймала
пол ЗА кромкой — на 117 мм ниже, и это высота стенда. Правда в том, что
камера на 658 мм над своим настилом против 716 по описанию. Знак у
сообщения детектора читается не с первого раза: ПЛЮС значит, что камера
НИЖЕ обещанного.

Линейкой подъёма над профилем не видно, и это не противоречие: меряется
крепление, а в описание идёт ОПТИЧЕСКИЙ ЦЕНТР, который при наклоне на 49
градусов уходит ниже верхней плоскости профиля.

Ошибка била по карте: настил уезжал на 58 мм вверх при
Grid/MaxGroundHeight 0.15, а шум глубины растёт как квадрат дальности и
на трёх метрах даёт около 40 мм — хвост перелезал порог, и настил местами
размечался как препятствие. После правки детектор печатает сдвиг +0 см.

Co-Authored-By: Claude Opus 5 <noreply@anthropic.com>

File: src/maze_nav/urdf/agro_robot_real.urdf.xacro (robot description, xacro)
@@ -919,13 +919,13 @@
        константой, не трогая вынос. -->
   <link name="camera_mount_link">
-    <visual><origin xyz="-0.0400 0 0" rpy="0 1.570796 0"/>
-      <geometry><cylinder radius="0.012" length="0.08"/></geometry>
+    <visual><origin xyz="-0.0150 0 0" rpy="0 1.570796 0"/>
+      <geometry><cylinder radius="0.012" length="0.03"/></geometry>
       <material name="hub"/></visual>
   </link>
   <joint name="camera_mount_joint" type="fixed">
     <parent link="base_link"/><child link="camera_mount_link"/>
-    <origin xyz="0.4905 0.0 0.6217"/>
-  </joint>
-  <!-- D435, наклон 50° вниз -->
+    <origin xyz="0.4405 0.0 0.5567"/>
+  </joint>
+  <!-- D435, наклон 49° вниз -->
   <link name="camera_link">
     <visual><geometry><box size="0.025 0.090 0.025"/></geometry>
@@ -934,5 +934,5 @@
   <joint name="camera_joint" type="fixed">
     <parent link="camera_mount_link"/><child link="camera_link"/>
-    <origin rpy="0 0.874410 0"/>
+    <origin rpy="0 0.855211 0"/>
   </joint>
   <!-- Стоит в начале base_link: центр колёсной базы на высоте оси.
